File: logic_board/logic_board.sch (KiCad schematic (older format))
At the start: 4 parts

Commit message: Use longer screws
The M2x6 screws are too short with the PCB in place. This requires upgrading to M2.3 screws.
Increased bore sizes. I had to make the top bosses tapered to accomodate the larger counterbore.
I tapered the bottom ones just to match.
Also increased the RELIEF to 0.8, as the parts do warp a bit and things stick during assembly.
Parts:
- H1, H2, H3, H4: footprint Mounting_Holes:MountingHole_2.2mm_M2_Pad -> MountingHole:MountingHole_2.5mm
Changed lines of the file:
@@
 F 0 "H1" H 1750 5196 50  0000 L CNN
 F 1 "MountingHole" H 1750 5105 50  0000 L CNN
-F 2 "Mounting_Holes:MountingHole_2.2mm_M2_Pad" H 1650 5150 50  0001 C CNN
+F 2 "MountingHole:MountingHole_2.5mm" H 1650 5150 50  0001 C CNN
 F 3 "~" H 1650 5150 50  0001 C CNN
 	1    1650 5150
@@
 F 0 "H2" H 1750 5496 50  0000 L CNN
 F 1 "MountingHole" H 1750 5405 50  0000 L CNN
-F 2 "Mounting_Holes:MountingHole_2.2mm_M2_Pad" H 1650 5450 50  0001 C CNN
+F 2 "MountingHole:MountingHole_2.5mm" H 1650 5450 50  0001 C CNN
 F 3 "~" H 1650 5450 50  0001 C CNN
 	1    1650 5450
@@
 F 0 "H3" H 1750 5796 50  0000 L CNN
 F 1 "MountingHole" H 1750 5705 50  0000 L CNN
-F 2 "Mounting_Holes:MountingHole_2.2mm_M2_Pad" H 1650 5750 50  0001 C CNN
+F 2 "MountingHole:MountingHole_2.5mm" H 1650 5750 50  0001 C CNN
 F 3 "~" H 1650 5750 50  0001 C CNN
 	1    1650 5750
@@
 F 0 "H4" H 1750 6096 50  0000 L CNN
 F 1 "MountingHole" H 1750 6005 50  0000 L CNN
-F 2 "Mounting_Holes:MountingHole_2.2mm_M2_Pad" H 1650 6050 50  0001 C CNN
+F 2 "MountingHole:MountingHole_2.5mm" H 1650 6050 50  0001 C CNN
 F 3 "~" H 1650 6050 50  0001 C CNN
 	1    1650 6050
