File: logic_board/audio.sch (KiCad schematic (older format))
At the start: 20 parts, among them J2 Audio In, J3 SJ2-3595X-SMT, U2 OPA340NA, U3 WM8731SEDS_V, Y2 12MHz

Commit message: Update to symbols from newest KiCad
LEDs were also on the wrong side of the board.
Parts:
- C10, C12, C15, C16, C17, C18, C19, C20: footprint Capacitors_SMD:C_0402 -> Capacitor_SMD:C_0402_1005Metric
- C13: footprint Capacitors_SMD:C_0805_HandSoldering -> Capacitor_SMD:C_0805_2012Metric_Pad1.15x1.40mm_HandSolder
- C23, C24: footprint Capacitors_SMD:C_1206_HandSoldering -> Capacitor_SMD:C_1206_3216Metric_Pad1.42x1.75mm_HandSolder
- R10, R7, R9: footprint Resistors_SMD:R_0402 -> Resistor_SMD:R_0402_1005Metric
- R6: footprint Resistors_SMD:R_0805_HandSoldering -> Resistor_SMD:R_0805_2012Metric_Pad1.15x1.40mm_HandSolder
- U2: footprint TO_SOT_Packages_SMD:TSOT-23-5_HandSoldering -> Package_TO_SOT_SMD:SOT-23-5_HandSoldering
- U3: footprint Housings_SSOP:SSOP-28_5.3x10.2mm_Pitch0.65mm -> Package_SO:SSOP-28_5.3x10.2mm_P0.65mm
Changed lines of the file:
@@
 F 0 "U3" H 5825 4137 60  0000 C CNN
 F 1 "WM8731SEDS_V" H 5825 4031 60  0000 C CNN
-F 2 "Housings_SSOP:SSOP-28_5.3x10.2mm_Pitch0.65mm" H 5800 1950 60  0001 C CNN
+F 2 "Package_SO:SSOP-28_5.3x10.2mm_P0.65mm" H 5800 1950 60  0001 C CNN
 F 3 "https://d3uzseaevmutz1.cloudfront.net/pubs/proDatasheet/WM8731_v4.9.pdf" H 5850 3050 60  0001 C CNN
 	1    5850 3050
@@
 F 0 "C12" V 2398 3950 50  0000 C CNN
 F 1 "0.1uF" V 2489 3950 50  0000 C CNN
-F 2 "Capacitors_SMD:C_0402" H 2688 3800 50  0001 C CNN
+F 2 "Capacitor_SMD:C_0402_1005Metric" H 2688 3800 50  0001 C CNN
 F 3 "~" H 2650 3950 50  0001 C CNN
 	1    2650 3950
@@
 F 0 "R6" V 3115 3950 50  0000 C CNN
 F 1 "50k" V 3206 3950 50  0000 C CNN
-F 2 "Resistors_SMD:R_0805_HandSoldering" V 2930 3950 50  0001 C CNN
+F 2 "Resistor_SMD:R_0805_2012Metric_Pad1.15x1.40mm_HandSolder" V 2930 3950 50  0001 C CNN
 F 3 "~" H 3000 3950 50  0001 C CNN
 	1    3000 3950
@@
 F 0 "R7" V 3443 4350 50  0000 C CNN
 F 1 "100k" V 3534 4350 50  0000 C CNN
-F 2 "Resistors_SMD:R_0402" V 3580 4350 50  0001 C CNN
+F 2 "Resistor_SMD:R_0402_1005Metric" V 3580 4350 50  0001 C CNN
 F 3 "~" H 3650 4350 50  0001 C CNN
 	1    3650 4350
@@
 F 0 "R9" H 8480 3696 50  0000 R CNN
 F 1 "47k" H 8480 3605 50  0000 R CNN
-F 2 "Resistors_SMD:R_0402" V 8480 3650 50  0001 C CNN
+F 2 "Resistor_SMD:R_0402_1005Metric" V 8480 3650 50  0001 C CNN
 F 3 "~" H 8550 3650 50  0001 C CNN
 	1    8550 3650
@@
 F 0 "R10" H 8770 3696 50  0000 L CNN
 F 1 "47k" H 8770 3605 50  0000 L CNN
-F 2 "Resistors_SMD:R_0402" V 8630 3650 50  0001 C CNN
+F 2 "Resistor_SMD:R_0402_1005Metric" V 8630 3650 50  0001 C CNN
 F 3 "~" H 8700 3650 50  0001 C CNN
 	1    8700 3650
@@
 F 0 "C18" V 3990 3850 50  0000 C CNN
 F 1 "0.1uF" V 3899 3850 50  0000 C CNN
-F 2 "Capacitors_SMD:C_0402" H 4188 3700 50  0001 C CNN
+F 2 "Capacitor_SMD:C_0402_1005Metric" H 4188 3700 50  0001 C CNN
 F 3 "~" H 4150 3850 50  0001 C CNN
 	1    4150 3850
@@
 F 0 "C15" H 3385 6496 50  0000 L CNN
 F 1 "0.1uF" H 3385 6405 50  0000 L CNN
-F 2 "Capacitors_SMD:C_0402" H 3308 6300 50  0001 C CNN
+F 2 "Capacitor_SMD:C_0402_1005Metric" H 3308 6300 50  0001 C CNN
 F 3 "~" H 3270 6450 50  0001 C CNN
 	1    3270 6450
@@
 F 0 "C17" H 3735 6496 50  0000 L CNN
 F 1 "0.1uF" H 3735 6405 50  0000 L CNN
-F 2 "Capacitors_SMD:C_0402" H 3658 6300 50  0001 C CNN
+F 2 "Capacitor_SMD:C_0402_1005Metric" H 3658 6300 50  0001 C CNN
 F 3 "~" H 3620 6450 50  0001 C CNN
 	1    3620 6450
@@
 F 0 "C19" H 4085 6496 50  0000 L CNN
 F 1 "0.1uF" H 4085 6405 50  0000 L CNN
-F 2 "Capacitors_SMD:C_0402" H 4008 6300 50  0001 C CNN
+F 2 "Capacitor_SMD:C_0402_1005Metric" H 4008 6300 50  0001 C CNN
 F 3 "~" H 3970 6450 50  0001 C CNN
 	1    3970 6450
@@
 F 0 "C13" H 3018 6496 50  0000 L CNN
 F 1 "10uF" H 3018 6405 50  0000 L CNN
-F 2 "Capacitors_SMD:C_0805_HandSoldering" H 2938 6300 50  0001 C CNN
+F 2 "Capacitor_SMD:C_0805_2012Metric_Pad1.15x1.40mm_HandSolder" H 2938 6300 50  0001 C CNN
 F 3 "~" H 2900 6450 50  0001 C CNN
 	1    2900 6450
@@
 F 0 "C16" H 4065 3546 50  0000 L CNN
 F 1 "0.1uF" H 4065 3455 50  0000 L CNN
-F 2 "Capacitors_SMD:C_0402" H 3988 3350 50  0001 C CNN
+F 2 "Capacitor_SMD:C_0402_1005Metric" H 3988 3350 50  0001 C CNN
 F 3 "~" H 3950 3500 50  0001 C CNN
 	1    3950 3500
@@
 F 0 "C20" H 4435 6496 50  0000 L CNN
 F 1 "0.1uF" H 4435 6405 50  0000 L CNN
-F 2 "Capacitors_SMD:C_0402" H 4358 6300 50  0001 C CNN
+F 2 "Capacitor_SMD:C_0402_1005Metric" H 4358 6300 50  0001 C CNN
 F 3 "~" H 4320 6450 50  0001 C CNN
 	1    4320 6450
@@
 F 0 "C23" V 8305 3250 50  0000 C CNN
 F 1 "220uF" V 8214 3250 50  0000 C CNN
-F 2 "Capacitors_SMD:C_1206_HandSoldering" H 8088 3100 50  0001 C CNN
+F 2 "Capacitor_SMD:C_1206_3216Metric_Pad1.42x1.75mm_HandSolder" H 8088 3100 50  0001 C CNN
 F 3 "~" H 8050 3250 50  0001 C CNN
 	1    8050 3250
@@
 F 0 "C24" V 8650 3350 50  0000 C CNN
 F 1 "220uF" V 8550 3350 50  0000 C CNN
-F 2 "Capacitors_SMD:C_1206_HandSoldering" H 8388 3200 50  0001 C CNN
+F 2 "Capacitor_SMD:C_1206_3216Metric_Pad1.42x1.75mm_HandSolder" H 8388 3200 50  0001 C CNN
 F 3 "~" H 8350 3350 50  0001 C CNN
 	1    8350 3350
@@
 F 0 "U2" H 3500 3850 50  0000 L CNN
 F 1 "OPA340NA" H 3500 3700 50  0000 L CNN
-F 2 "TO_SOT_Packages_SMD:TSOT-23-5_HandSoldering" H 3450 3650 50  0001 L CNN
+F 2 "Package_TO_SOT_SMD:SOT-23-5_HandSoldering" H 3450 3650 50  0001 L CNN
 F 3 "http://www.ti.com/lit/ds/symlink/opa340.pdf" H 3550 4050 50  0001 C CNN
 	1    3550 3850
@@
 F 0 "C10" H 4835 6496 50  0000 L CNN
 F 1 "0.1uF" H 4835 6405 50  0000 L CNN
-F 2 "Capacitors_SMD:C_0402" H 4758 6300 50  0001 C CNN
+F 2 "Capacitor_SMD:C_0402_1005Metric" H 4758 6300 50  0001 C CNN
 F 3 "~" H 4720 6450 50  0001 C CNN
 	1    4720 6450

Commit message: Update all 0402 SMD packages to 0603
Mainly to make soldering easier. 0402 was unnecessarily small.
Parts:
- C10, C12, C15, C16, C17, C18, C19, C20: footprint Capacitor_SMD:C_0402_1005Metric -> Capacitor_SMD:C_0603_1608Metric_Pad1.05x0.95mm_HandSolder
- R10, R7, R9: footprint Resistor_SMD:R_0402_1005Metric -> Resistor_SMD:R_0603_1608Metric_Pad1.05x0.95mm_HandSolder
Changed lines of the file:
@@
 F 0 "C12" V 2398 3950 50  0000 C CNN
 F 1 "0.1uF" V 2489 3950 50  0000 C CNN
-F 2 "Capacitor_SMD:C_0402_1005Metric" H 2688 3800 50  0001 C CNN
+F 2 "Capacitor_SMD:C_0603_1608Metric_Pad1.05x0.95mm_HandSolder" H 2688 3800 50  0001 C CNN
 F 3 "~" H 2650 3950 50  0001 C CNN
 	1    2650 3950
@@
 F 0 "R7" V 3443 4350 50  0000 C CNN
 F 1 "100k" V 3534 4350 50  0000 C CNN
-F 2 "Resistor_SMD:R_0402_1005Metric" V 3580 4350 50  0001 C CNN
+F 2 "Resistor_SMD:R_0603_1608Metric_Pad1.05x0.95mm_HandSolder" V 3580 4350 50  0001 C CNN
 F 3 "~" H 3650 4350 50  0001 C CNN
 	1    3650 4350
@@
 F 0 "R9" H 8480 3696 50  0000 R CNN
 F 1 "47k" H 8480 3605 50  0000 R CNN
-F 2 "Resistor_SMD:R_0402_1005Metric" V 8480 3650 50  0001 C CNN
+F 2 "Resistor_SMD:R_0603_1608Metric_Pad1.05x0.95mm_HandSolder" V 8480 3650 50  0001 C CNN
 F 3 "~" H 8550 3650 50  0001 C CNN
 	1    8550 3650
@@
 F 0 "R10" H 8770 3696 50  0000 L CNN
 F 1 "47k" H 8770 3605 50  0000 L CNN
-F 2 "Resistor_SMD:R_0402_1005Metric" V 8630 3650 50  0001 C CNN
+F 2 "Resistor_SMD:R_0603_1608Metric_Pad1.05x0.95mm_HandSolder" V 8630 3650 50  0001 C CNN
 F 3 "~" H 8700 3650 50  0001 C CNN
 	1    8700 3650
@@
 F 0 "C18" V 3990 3850 50  0000 C CNN
 F 1 "0.1uF" V 3899 3850 50  0000 C CNN
-F 2 "Capacitor_SMD:C_0402_1005Metric" H 4188 3700 50  0001 C CNN
+F 2 "Capacitor_SMD:C_0603_1608Metric_Pad1.05x0.95mm_HandSolder" H 4188 3700 50  0001 C CNN
 F 3 "~" H 4150 3850 50  0001 C CNN
 	1    4150 3850
@@
 F 0 "C15" H 3385 6496 50  0000 L CNN
 F 1 "0.1uF" H 3385 6405 50  0000 L CNN
-F 2 "Capacitor_SMD:C_0402_1005Metric" H 3308 6300 50  0001 C CNN
+F 2 "Capacitor_SMD:C_0603_1608Metric_Pad1.05x0.95mm_HandSolder" H 3308 6300 50  0001 C CNN
 F 3 "~" H 3270 6450 50  0001 C CNN
 	1    3270 6450
@@
 F 0 "C17" H 3735 6496 50  0000 L CNN
 F 1 "0.1uF" H 3735 6405 50  0000 L CNN
-F 2 "Capacitor_SMD:C_0402_1005Metric" H 3658 6300 50  0001 C CNN
+F 2 "Capacitor_SMD:C_0603_1608Metric_Pad1.05x0.95mm_HandSolder" H 3658 6300 50  0001 C CNN
 F 3 "~" H 3620 6450 50  0001 C CNN
 	1    3620 6450
@@
 F 0 "C19" H 4085 6496 50  0000 L CNN
 F 1 "0.1uF" H 4085 6405 50  0000 L CNN
-F 2 "Capacitor_SMD:C_0402_1005Metric" H 4008 6300 50  0001 C CNN
+F 2 "Capacitor_SMD:C_0603_1608Metric_Pad1.05x0.95mm_HandSolder" H 4008 6300 50  0001 C CNN
 F 3 "~" H 3970 6450 50  0001 C CNN
 	1    3970 6450
@@
 F 0 "C16" H 4065 3546 50  0000 L CNN
 F 1 "0.1uF" H 4065 3455 50  0000 L CNN
-F 2 "Capacitor_SMD:C_0402_1005Metric" H 3988 3350 50  0001 C CNN
+F 2 "Capacitor_SMD:C_0603_1608Metric_Pad1.05x0.95mm_HandSolder" H 3988 3350 50  0001 C CNN
 F 3 "~" H 3950 3500 50  0001 C CNN
 	1    3950 3500
@@
 F 0 "C20" H 4435 6496 50  0000 L CNN
 F 1 "0.1uF" H 4435 6405 50  0000 L CNN
-F 2 "Capacitor_SMD:C_0402_1005Metric" H 4358 6300 50  0001 C CNN
+F 2 "Capacitor_SMD:C_0603_1608Metric_Pad1.05x0.95mm_HandSolder" H 4358 6300 50  0001 C CNN
 F 3 "~" H 4320 6450 50  0001 C CNN
 	1    4320 6450
@@
 F 0 "C10" H 4835 6496 50  0000 L CNN
 F 1 "0.1uF" H 4835 6405 50  0000 L CNN
-F 2 "Capacitor_SMD:C_0402_1005Metric" H 4758 6300 50  0001 C CNN
+F 2 "Capacitor_SMD:C_0603_1608Metric_Pad1.05x0.95mm_HandSolder" H 4758 6300 50  0001 C CNN
 F 3 "~" H 4720 6450 50  0001 C CNN
 	1    4720 6450
