File: logic_board/mcu.kicad_sch (KiCad schematic)
At the start: 31 parts, among them J2 SOICBite, SW1 SW_Push, SW2 SW_Push, SW3 SW_Push, SW4 SW_Push, U1 STM32H7B0RBTx, Y1 8Mhz

Commit message: Fix JLCPCB issues
- Use fabrication toolkit plugin to fix compnent orientations.
- Add part numbers to all components
- Manually fix some footprint rotation issues and incorrect origins.
Parts:
- C1, C2: LCSC Part Number (none) -> C1648
- C17, C18, C19, C20, C21, C22, C30: footprint Capacitor_SMD:C_0402_1005Metric -> Capacitor_SMD:C_0603_1608Metric; LCSC Part Number (none) -> C14663
- C27, C28: LCSC Part Number (none) -> C23630
- C29: footprint Capacitor_SMD:C_0603_1608Metric -> Capacitor_SMD:C_0805_2012Metric; LCSC Part Number (none) -> C15850
- CR1, CR2: FT Rotation Offset (none) -> -90
- D1: now left out of the parts list
- R19, R20: LCSC Part Number (none) -> C23350
- R2, R24: LCSC Part Number (none) -> C25804
- R21, R22, R3: LCSC Part Number (none) -> C21190
Changed lines of the file:
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@@
 			)
 		)
-		(property "Footprint" "Capacitor_SMD:C_0402_1005Metric"
+		(property "Footprint" "Capacitor_SMD:C_0603_1608Metric"
 			(at 125.4252 165.1 0)
 			(effects
@@
 			)
 		)
-		(property "LCSC part number" ""
+		(property "LCSC Part Number" "C14663"
 			(at 124.46 161.29 0)
 			(effects
@@
 			)
 		)
-		(property "LCSC part number" ""
+		(property "LCSC Part Number" "C23630"
 			(at 101.6 110.49 0)
 			(effects
@@
 			)
 		)
-		(property "LCSC part number" ""
+		(property "LCSC Part Number" "C25804"
 			(at 185.42 76.2 0)
 			(effects
@@
 			)
 		)
-		(property "Footprint" "Capacitor_SMD:C_0402_1005Metric"
+		(property "Footprint" "Capacitor_SMD:C_0603_1608Metric"
 			(at 136.8552 165.1 0)
 			(effects
@@
 			)
 		)
-		(property "LCSC part number" ""
+		(property "LCSC Part Number" "C14663"
 			(at 135.89 161.29 0)
 			(effects
@@
 			)
 		)
-		(property "LCSC part number" ""
-			(at 218.44 30.48 90)
-			(effects
-				(font
-					(size 1.27 1.27)
-				)
-				(hide yes)
-			)
-		)
 		(pin "5"
 		)
@@
 			)
 		)
-		(property "LCSC part number" ""
-			(at 78.74 54.61 0)
-			(effects
-				(font
-					(size 1.27 1.27)
-				)
-				(hide yes)
-			)
-		)
 		(pin "2"
 		)
@@
 			)
 		)
-		(property "Footprint" "Capacitor_SMD:C_0402_1005Metric"
+		(property "Footprint" "Capacitor_SMD:C_0603_1608Metric"
 			(at 113.9952 165.1 0)
 			(effects
@@
 			)
 		)
-		(property "LCSC part number" ""
+		(property "LCSC Part Number" "C14663"
 			(at 113.03 161.29 0)
 			(effects
@@
 			)
 		)
-		(property "Footprint" "Capacitor_SMD:C_0402_1005Metric"
+		(property "Footprint" "Capacitor_SMD:C_0603_1608Metric"
 			(at 102.5652 165.1 0)
 			(effects
@@
 			)
 		)
-		(property "LCSC part number" ""
+		(property "LCSC Part Number" "C14663"
 			(at 101.6 161.29 0)
 			(effects
@@
 			)
 		)
-		(property "LCSC part number" ""
+		(property "LCSC Part Number" "C21190"
 			(at 152.4 74.93 90)
 			(effects
@@
 			)
 		)
-		(property "LCSC part number" ""
+		(property "FT Rotation Offset" "-90"
 			(at 240.03 60.96 0)
 			(effects
@@
 			)
 		)
-		(property "LCSC part number" ""
+		(property "LCSC Part Number" "C21190"
 			(at 172.72 99.06 0)
 			(effects
@@
 		(unit 1)
 		(exclude_from_sim no)
-		(in_bom yes)
+		(in_bom no)
 		(on_board yes)
 		(dnp no)
@@
 			)
 		)
-		(property "LCSC part number" ""
-			(at 207.01 137.16 0)
-			(effects
-				(font
-					(size 1.27 1.27)
-				)
-				(hide yes)
-			)
-		)
 		(pin "1"
 		)
@@
 			)
 		)
-		(property "LCSC part number" ""
-			(at 128.27 77.47 0)
-			(effects
-				(font
-					(size 1.27 1.27)
-				)
-				(hide yes)
-			)
-		)
 		(pin "38"
 		)
@@
 			)
 		)
-		(property "LCSC part number" ""
+		(property "LCSC Part Number" "C1648"
 			(at 86.36 59.69 0)
 			(effects
@@
 			)
 		)
-		(property "LCSC part number" ""
-			(at 46.99 171.45 0)
-			(effects
-				(font
-					(size 1.27 1.27)
-				)
-				(hide yes)
-			)
-		)
 		(pin "1"
 		)
@@
 			)
 		)
-		(property "Footprint" "Capacitor_SMD:C_0402_1005Metric"
+		(property "Footprint" "Capacitor_SMD:C_0603_1608Metric"
 			(at 148.2852 165.1 0)
 			(effects
@@
 			)
 		)
-		(property "LCSC part number" ""
+		(property "LCSC Part Number" "C14663"
 			(at 147.32 161.29 0)
 			(effects
@@
 			)
 		)
-		(property "LCSC part number" ""
+		(property "LCSC Part Number" "C21190"
 			(at 175.26 99.06 0)
 			(effects
@@
 			)
 		)
-		(property "LCSC part number" ""
+		(property "LCSC Part Number" "C23350"
 			(at 190.5 134.62 90)
 			(effects
@@
 			)
 		)
-		(property "LCSC part number" ""
+		(property "LCSC Part Number" "C23630"
 			(at 95.25 110.49 0)
 			(effects
@@
 			)
 		)
-		(property "Footprint" "Capacitor_SMD:C_0402_1005Metric"
+		(property "Footprint" "Capacitor_SMD:C_0603_1608Metric"
 			(at 59.3852 46.99 0)
 			(effects
@@
 			)
 		)
-		(property "LCSC part number" ""
+		(property "LCSC Part Number" "C14663"
 			(at 58.42 43.18 0)
 			(effects
@@
 			)
 		)
-		(property "LCSC part number" ""
+		(property "LCSC Part Number" "C25804"
 			(at 102.87 41.91 90)
 			(effects
@@
 			)
 		)
-		(property "LCSC part number" ""
-			(at 46.99 147.32 0)
-			(effects
-				(font
-					(size 1.27 1.27)
-				)
-				(hide yes)
-			)
-		)
 		(pin "1"
 		)
@@
 			)
 		)
-		(property "LCSC part number" ""
-			(at 218.44 44.45 90)
-			(effects
-				(font
-					(size 1.27 1.27)
-				)
-				(hide yes)
-			)
-		)
 		(pin "5"
 		)
@@
 			)
 		)
-		(property "LCSC part number" ""
+		(property "FT Rotation Offset" "-90"
 			(at 240.03 100.33 0)
 			(effects
@@
 			)
 		)
-		(property "LCSC part number" ""
-			(at 255.27 35.56 0)
-			(effects
-				(font
-					(size 1.27 1.27)
-				)
-				(hide yes)
-			)
-		)
 		(pin "8"
 		)
@@
 			)
 		)
-		(property "Footprint" "Capacitor_SMD:C_0402_1005Metric"
+		(property "Footprint" "Capacitor_SMD:C_0603_1608Metric"
 			(at 91.1352 165.1 0)
 			(effects
@@
 			)
 		)
-		(property "LCSC part number" ""
+		(property "LCSC Part Number" "C14663"
 			(at 90.17 161.29 0)
 			(effects
@@
 			)
 		)
-		(property "LCSC part number" ""
-			(at 46.99 134.62 0)
-			(effects
-				(font
-					(size 1.27 1.27)
-				)
-				(hide yes)
-			)
-		)
 		(pin "1"
 		)
@@
 			)
 		)
-		(property "LCSC part number" ""
+		(property "LCSC Part Number" "C23350"
 			(at 190.5 139.7 90)
 			(effects
@@
 			)
 		)
-		(property "LCSC part number" ""
+		(property "LCSC Part Number" "C1648"
 			(at 69.85 59.69 0)
 			(effects
@@
 			)
 		)
-		(property "LCSC part number" ""
-			(at 46.99 160.02 0)
-			(effects
-				(font
-					(size 1.27 1.27)
-				)
-				(hide yes)
-			)
-		)
 		(pin "1"
 		)
@@
 			)
 		)
-		(property "Footprint" "Capacitor_SMD:C_0603_1608Metric"
+		(property "Footprint" "Capacitor_SMD:C_0805_2012Metric"
 			(at 160.9852 165.1 0)
 			(effects
@@
 			)
 		)
-		(property "LCSC part number" ""
+		(property "LCSC Part Number" "C15850"
 			(at 160.02 161.29 0)
 			(effects

Commit message: Standardize part values and flesh out documentation.
Parts:
- R21, R22: value 1k -> 10k; LCSC Part Number C21190 -> C25804
Other:
- moved on the sheet: C1, C2, Y1
Changed lines of the file:
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@@
 	)
 	(junction
-		(at 69.85 54.61)
+		(at 72.39 58.42)
 		(diameter 0)
 		(color 0 0 0 0)
@@
 	)
 	(junction
-		(at 86.36 54.61)
+		(at 88.9 58.42)
 		(diameter 0)
 		(color 0 0 0 0)
@@
 	)
 	(junction
-		(at 86.36 64.77)
+		(at 88.9 68.58)
 		(diameter 0)
 		(color 0 0 0 0)
@@
 	(wire
 		(pts
-			(xy 69.85 64.77) (xy 86.36 64.77)
+			(xy 72.39 68.58) (xy 88.9 68.58)
 		)
 		(stroke
@@
 	(wire
 		(pts
+			(xy 88.9 49.53) (xy 110.49 49.53)
+		)
+		(stroke
+			(width 0)
+			(type default)
+		)
+	)
+	(wire
+		(pts
 			(xy 217.17 137.16) (xy 217.17 142.24)
 		)
@@
 	(wire
 		(pts
-			(xy 86.36 63.5) (xy 86.36 64.77)
+			(xy 88.9 67.31) (xy 88.9 68.58)
 		)
 		(stroke
@@
 	(wire
 		(pts
-			(xy 69.85 46.99) (xy 69.85 54.61)
+			(xy 72.39 46.99) (xy 72.39 58.42)
 		)
 		(stroke
@@
 	(wire
 		(pts
-			(xy 69.85 54.61) (xy 74.93 54.61)
+			(xy 72.39 58.42) (xy 77.47 58.42)
 		)
 		(stroke
@@
 	(wire
 		(pts
-			(xy 86.36 67.31) (xy 86.36 64.77)
+			(xy 88.9 71.12) (xy 88.9 68.58)
 		)
 		(stroke
@@
 	(wire
 		(pts
-			(xy 86.36 54.61) (xy 86.36 55.88)
+			(xy 88.9 58.42) (xy 88.9 59.69)
 		)
 		(stroke
@@
 	(wire
 		(pts
-			(xy 86.36 54.61) (xy 82.55 54.61)
+			(xy 88.9 58.42) (xy 85.09 58.42)
 		)
 		(stroke
@@
 	(wire
 		(pts
-			(xy 86.36 49.53) (xy 86.36 54.61)
+			(xy 88.9 49.53) (xy 88.9 58.42)
 		)
 		(stroke
@@
 	(wire
 		(pts
+			(xy 72.39 46.99) (xy 110.49 46.99)
+		)
+		(stroke
+			(width 0)
+			(type default)
+		)
+	)
+	(wire
+		(pts
 			(xy 146.05 113.03) (xy 175.26 113.03)
 		)
@@
 	(wire
 		(pts
-			(xy 69.85 54.61) (xy 69.85 55.88)
+			(xy 72.39 58.42) (xy 72.39 59.69)
 		)
 		(stroke
@@
 	(wire
 		(pts
-			(xy 110.49 49.53) (xy 86.36 49.53)
-		)
-		(stroke
-			(width 0)
-			(type default)
-		)
-	)
-	(wire
-		(pts
 			(xy 90.17 152.4) (xy 90.17 153.67)
 		)
@@
 	(wire
 		(pts
-			(xy 110.49 46.99) (xy 69.85 46.99)
-		)
-		(stroke
-			(width 0)
-			(type default)
-		)
-	)
-	(wire
-		(pts
 			(xy 229.87 43.18) (xy 250.19 43.18)
 		)
@@
 	(wire
 		(pts
-			(xy 69.85 64.77) (xy 69.85 63.5)
+			(xy 72.39 68.58) (xy 72.39 67.31)
 		)
 		(stroke
@@
 	(symbol
 		(lib_id "Device:Crystal")
-		(at 78.74 54.61 0)
+		(at 81.28 58.42 0)
 		(unit 1)
 		(exclude_from_sim no)
@@
 		(fields_autoplaced yes)
 		(property "Reference" "Y1"
-			(at 78.74 46.99 0)
+			(at 81.28 50.8 0)
 			(effects
 				(font
@@
 		)
 		(property "Value" "8Mhz"
-			(at 78.74 49.53 0)
+			(at 81.28 53.34 0)
 			(effects
 				(font
@@
 		)
 		(property "Footprint" "Crystal:Crystal_SMD_5032-2Pin_5.0x3.2mm"
-			(at 78.74 54.61 0)
+			(at 81.28 58.42 0)
 			(effects
 				(font
@@
 		)
 		(property "Datasheet" "~"
-			(at 78.74 54.61 0)
+			(at 81.28 58.42 0)
 			(effects
 				(font
@@
 		)
 		(property "Description" "Two pin crystal"
-			(at 78.74 54.61 0)
+			(at 81.28 58.42 0)
 			(effects
 				(font
@@
 		)
 		(property "LCSC Part Number" "C115962"
-			(at 78.74 54.61 0)
+			(at 81.28 58.42 0)
 			(effects
 				(font
@@
 			)
 		)
-		(property "Value" "1k"
+		(property "Value" "10k"
 			(at 170.18 100.3299 0)
 			(effects
@@
 			)
 		)
-		(property "LCSC Part Number" "C21190"
+		(property "LCSC Part Number" "C25804"
 			(at 172.72 99.06 0)
 			(effects
@@
 	(symbol
 		(lib_id "Device:C")
-		(at 86.36 59.69 0)
+		(at 88.9 63.5 0)
 		(unit 1)
 		(exclude_from_sim no)
@@
 		(fields_autoplaced yes)
 		(property "Reference" "C2"
-			(at 90.17 58.4199 0)
+			(at 92.71 62.2299 0)
 			(effects
 				(font
@@
 		)
 		(property "Value" "20pF"
-			(at 90.17 60.9599 0)
+			(at 92.71 64.7699 0)
 			(effects
 				(font
@@
 		)
 		(property "Footprint" "Capacitor_SMD:C_0603_1608Metric"
-			(at 87.3252 63.5 0)
+			(at 89.8652 67.31 0)
 			(effects
 				(font
@@
 		)
 		(property "Datasheet" "~"
-			(at 86.36 59.69 0)
+			(at 88.9 63.5 0)
 			(effects
 				(font
@@
 		)
 		(property "Description" "Unpolarized capacitor"
-			(at 86.36 59.69 0)
+			(at 88.9 63.5 0)
 			(effects
 				(font
@@
 		)
 		(property "LCSC Part Number" "C1648"
-			(at 86.36 59.69 0)
+			(at 88.9 63.5 0)
 			(effects
 				(font
@@
 			)
 		)
-		(property "Value" "1k"
+		(property "Value" "10k"
 			(at 177.8 100.3299 0)
 			(effects
@@
 			)
 		)
-		(property "LCSC Part Number" "C21190"
+		(property "LCSC Part Number" "C25804"
 			(at 175.26 99.06 0)
 			(effects
@@
 	(symbol
 		(lib_id "Device:C")
-		(at 69.85 59.69 0)
+		(at 72.39 63.5 0)
 		(unit 1)
 		(exclude_from_sim no)
@@
 		(dnp no)
 		(property "Reference" "C1"
-			(at 64.008 58.42 0)
+			(at 66.548 62.23 0)
 			(effects
 				(font
@@
 		)
 		(property "Value" "20pF"
-			(at 62.484 61.214 0)
+			(at 65.024 65.024 0)
 			(effects
 				(font
@@
 		)
 		(property "Footprint" "Capacitor_SMD:C_0603_1608Metric"
-			(at 70.8152 63.5 0)
+			(at 73.3552 67.31 0)
 			(effects
 				(font
@@
 		)
 		(property "Datasheet" "~"
-			(at 69.85 59.69 0)
+			(at 72.39 63.5 0)
 			(effects
 				(font
@@
 		)
 		(property "Description" "Unpolarized capacitor"
-			(at 69.85 59.69 0)
+			(at 72.39 63.5 0)
 			(effects
 				(font
@@
 		)
 		(property "LCSC Part Number" "C1648"
-			(at 69.85 59.69 0)
+			(at 72.39 63.5 0)
 			(effects
 				(font
@@
 	(symbol
 		(lib_id "power:GND")
-		(at 86.36 67.31 0)
+		(at 88.9 71.12 0)
 		(unit 1)
 		(exclude_from_sim no)
@@
 		(fields_autoplaced yes)
 		(property "Reference" "#PWR01"
-			(at 86.36 73.66 0)
+			(at 88.9 77.47 0)
 			(effects
 				(font
@@
 		)
 		(property "Value" "GND"
-			(at 86.36 72.39 0)
+			(at 88.9 76.2 0)
 			(effects
 				(font
@@
 		)
 		(property "Footprint" ""
-			(at 86.36 67.31 0)
+			(at 88.9 71.12 0)
 			(effects
 				(font
@@
 		)
 		(property "Datasheet" ""
-			(at 86.36 67.31 0)
+			(at 88.9 71.12 0)
 			(effects
 				(font
@@
 		)
 		(property "Description" "Power symbol creates a global label with name \"GND\" , ground"
-			(at 86.36 67.31 0)
+			(at 88.9 71.12 0)
 			(effects
 				(font
