File: logic_board/Power.kicad_sch (KiCad schematic)
At the start: 25 parts, among them J3 USB_C_Receptacle_USB2.0_16P, J5 Battery, Q1 BSS138, SW5 SW_SPDT, U3 BQ25185DLHR, U5 USBLC6-2SC6, U7 TLV62568ADRL

Commit message: Minor cosmetic tweaks, fix silkscreen references
Other:
- title: (none) -> Power, Regulators, Charging
Changed lines of the file:
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@@
 	(generator_version "9.0")
 	(paper "A4")
+	(title_block
+		(title "Power, Regulators, Charging")
+		(date "2026-01-02")
+		(rev "2.0")
+	)
 	(text "Max charge current/\ninput current: 400mA"
 		(exclude_from_sim no)
