File: logic_board/codec.kicad_sch (KiCad schematic)
At the start: 39 parts, among them J1 SJ3-35083C-TR, J4 Conn_01x02, U2 ES8388, U6 TLV9061xDBV

Commit message: Minor cosmetic tweaks, fix silkscreen references
Other:
- title: (none) -> Audio Codec/Amplifiers
Changed lines of the file:
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@@
 	(generator_version "9.0")
 	(paper "A4")
+	(title_block
+		(title "Audio Codec/Amplifiers")
+		(date "2026-01-02")
+		(rev "2.0")
+	)
 	(text "Headphone Output"
 		(exclude_from_sim no)
